File: mic_base/mic_base.kicad_pcb (KiCad board)
At the start: 2 copper layers, 0 parts

Commit message: basically done, maybe add some finishing touches later
Parts:
- added C1: 22uF, Capacitor_THT:C_Disc_D7.5mm_W2.5mm_P5.00mm, F.Cu at (93.5, 73.0)
- added C2: 22uF, Capacitor_THT:C_Disc_D7.5mm_W2.5mm_P5.00mm, F.Cu at (98.5, 81.5)
- added C3: 22uF, Capacitor_THT:C_Disc_D7.5mm_W2.5mm_P5.00mm, F.Cu at (93.5, 87.5)
- added C4: 2200uF, Capacitor_THT:CP_Radial_D10.0mm_P5.00mm, F.Cu at (122.0, 60.5)
- added C5: 2200uF, Capacitor_THT:CP_Radial_D10.0mm_P5.00mm, F.Cu at (122.0, 67.5)
- added C6: 2200uF, Capacitor_THT:CP_Radial_D10.0mm_P5.00mm, F.Cu at (87.0, 63.0)
- added C7: 2200uF, Capacitor_THT:CP_Radial_D10.0mm_P5.00mm, F.Cu at (98.0, 63.0)
- added H1: MountingHole_Pad, MountingHole:MountingHole_2.2mm_M2_DIN965_Pad, F.Cu at (82.0, 47.5)
- added H2: MountingHole_Pad, MountingHole:MountingHole_2.2mm_M2_DIN965_Pad, F.Cu at (125.5, 47.5)
- added H3: MountingHole_Pad, MountingHole:MountingHole_2.2mm_M2_DIN965_Pad, F.Cu at (82.0, 91.0)
- added H4: MountingHole_Pad, MountingHole:MountingHole_2.2mm_M2_DIN965_Pad, F.Cu at (125.5, 91.0)
- added IC1: 1512P08-U, Footprints:DIP781W46P254L952H432Q8N, F.Cu at (112.5, 84.0)
- added J1: +Power-, Connector_JST:JST_XH_B2B-XH-A_1x02_P2.50mm_Vertical, F.Cu at (87.0, 53.0)
- added J2: +Out-, Connector_JST:JST_XH_B2B-XH-A_1x02_P2.50mm_Vertical, F.Cu at (87.3, 86.0)
- added J3: -Gain+, Connector_JST:JST_XH_B2B-XH-A_1x02_P2.50mm_Vertical, F.Cu at (113.5, 76.0)
- added J4: +Mic In-, Connector_JST:JST_XH_B3B-XH-A_1x03_P2.50mm_Vertical, F.Cu at (87.3, 77.0)
- added R1: 2.2k, PCM_Resistor_THT_AKL:R_Axial_DIN0204_L3.6mm_D1.6mm_P7.62mm_Horizontal, F.Cu at (92.7, 84.5)
- added R2: 2.2k, PCM_Resistor_THT_AKL:R_Axial_DIN0204_L3.6mm_D1.6mm_P7.62mm_Horizontal, F.Cu at (115.0, 59.4)
- added R3: 2.2k, PCM_Resistor_THT_AKL:R_Axial_DIN0204_L3.6mm_D1.6mm_P7.62mm_Horizontal, F.Cu at (100.3, 78.5)
- added R4: 2.2k, PCM_Resistor_THT_AKL:R_Axial_DIN0204_L3.6mm_D1.6mm_P7.62mm_Horizontal, F.Cu at (107.5, 59.4)
- added R5: 100, PCM_Resistor_THT_AKL:R_Axial_DIN0204_L3.6mm_D1.6mm_P7.62mm_Horizontal, F.Cu at (110.0, 67.0)
- added R6: 100, PCM_Resistor_THT_AKL:R_Axial_DIN0204_L3.6mm_D1.6mm_P7.62mm_Horizontal, F.Cu at (112.5, 67.0)
- added R7: 3.9k, PCM_Resistor_THT_AKL:R_Axial_DIN0204_L3.6mm_D1.6mm_P7.62mm_Horizontal, F.Cu at (100.3, 76.0)
- added R8: 3.9k, PCM_Resistor_THT_AKL:R_Axial_DIN0204_L3.6mm_D1.6mm_P7.62mm_Horizontal, F.Cu at (92.7, 70.0)
- added U1: NMA0515SC, Converter_DCDC:Converter_DCDC_Murata_NMAxxxxSC_THT, F.Cu at (95.5, 52.0)
Routing:
- net /-VOut: track 0.00 -> 60.5 mm
- net /+VOut: track 0.00 -> 52.3 mm
- net /AGND: track 0.00 -> 38.6 mm
- net /+5: track 0.00 -> 32.7 mm
- net Net-(IC1--IN): track 0.00 -> 24.1 mm
- net Net-(IC1-OUT): track 0.00 -> 22.8 mm
- net Net-(IC1-+IN): track 0.00 -> 19.7 mm
- net /-Mic: track 0.00 -> 15.0 mm
- net Net-(U1-VOUT-): track 0.00 -> 12.6 mm
- net /+Mic: track 0.00 -> 10.7 mm
- net Net-(U1-VOUT+): track 0.00 -> 9.18 mm
- net /+Gain: track 0.00 -> 6.40 mm
- net /Out: track 0.00 -> 6.07 mm
- net /-Gain: track 0.00 -> 5.90 mm
- added copper zone on B.Cu, net /GND
Other:
- board outline added: 50 x 50 mm
- board text added: "1/1"
- board text added: "Hi-Fi Mic Base"
