File: mic_base/mic_base.kicad_sch (KiCad schematic)
At the start: 20 parts, among them IC1 1512P08-U, J1 +Power-, J2 +Out-, J3 +Gain-, J4 +Mic In-, U1 NMA0515SC

Commit message: basically done, maybe add some finishing touches later
Parts:
- added C7: 2200uF, Capacitor_THT:CP_Radial_D10.0mm_P5.00mm, symbol Device:C_Polarized_Small
- added H1, H2, H3, H4: MountingHole_Pad, MountingHole:MountingHole_2.2mm_M2_DIN965_Pad, symbol Mechanical:MountingHole_Pad
- J3: value +Gain- -> -Gain+
- R1, R2, R3, R4, R5, R6, R7, R8: footprint PCM_Resistor_THT_AKL:R_Axial_DIN0207_L6.3mm_D2.5mm_P10.16mm_Horizontal -> PCM_Resistor_THT_AKL:R_Axial_DIN0204_L3.6mm_D1.6mm_P7.62mm_Horizontal
Connections:
- net +5: now also C7.1
- net GND: now also H1.1, H2.1, H3.1, H4.1
- net PGND renamed AGND
- net AGND: now also C7.2
Other:
- note added: "1"
- note added: "Hi-Fi Mic Base"
- note added: "Layout"
- moved on the sheet: C1, C2, C3, C4, C5, C6, IC1, J1, J2, J3, J4, R1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

Commit message: moved capacitors, made pcb smaller
Connections:
- net +VOut: no longer C5.1
- net -VOut: no longer C4.1
- net at R6.2, U1.6 (VOUT+): now also C5.1
- net at R5.2, U1.4 (VOUT-): now also C4.1
Other:
- moved on the sheet: C4, C5, R5, R6
Changed lines of the file:
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@@
 	)
 	(junction
-		(at 80.01 46.99)
+		(at 116.84 36.83)
 		(diameter 0)
 		(color 0 0 0 0)
 	)
 	(junction
-		(at 85.09 83.82)
+		(at 80.01 46.99)
 		(diameter 0)
 		(color 0 0 0 0)
 	)
 	(junction
-		(at 156.21 68.58)
+		(at 85.09 83.82)
 		(diameter 0)
 		(color 0 0 0 0)
 	)
 	(junction
-		(at 125.73 41.91)
+		(at 156.21 68.58)
 		(diameter 0)
 		(color 0 0 0 0)
@@
 	)
 	(junction
-		(at 125.73 46.99)
+		(at 116.84 41.91)
 		(diameter 0)
 		(color 0 0 0 0)
 	)
 	(junction
-		(at 125.73 36.83)
+		(at 116.84 46.99)
 		(diameter 0)
 		(color 0 0 0 0)
@@
 	(wire
 		(pts
-			(xy 130.81 46.99) (xy 125.73 46.99)
-		)
-		(stroke
-			(width 0)
-			(type default)
-			(color 0 160 255 1)
-		)
-	)
-	(wire
-		(pts
 			(xy 135.89 71.12) (xy 135.89 62.23)
 		)
@@
 	(wire
 		(pts
-			(xy 125.73 36.83) (xy 130.81 36.83)
-		)
-		(stroke
-			(width 0)
-			(type default)
-			(color 255 0 0 1)
-		)
-	)
-	(wire
-		(pts
 			(xy 156.21 78.74) (xy 158.75 78.74)
 		)
@@
 	(wire
 		(pts
-			(xy 78.74 91.44) (xy 72.39 91.44)
+			(xy 116.84 41.91) (xy 130.81 41.91)
 		)
 		(stroke
 			(width 0)
 			(type default)
+			(color 0 160 255 1)
 		)
 	)
 	(wire
 		(pts
-			(xy 130.81 69.85) (xy 130.81 71.12)
+			(xy 78.74 91.44) (xy 72.39 91.44)
 		)
 		(stroke
@@
 	(wire
 		(pts
-			(xy 114.3 41.91) (xy 125.73 41.91)
+			(xy 130.81 69.85) (xy 130.81 71.12)
 		)
 		(stroke
 			(width 0)
 			(type default)
-			(color 0 160 255 1)
 		)
 	)
 	(wire
 		(pts
-			(xy 156.21 50.8) (xy 160.02 50.8)
+			(xy 114.3 41.91) (xy 116.84 41.91)
 		)
 		(stroke
 			(width 0)
 			(type default)
+			(color 0 160 255 1)
 		)
 	)
 	(wire
 		(pts
-			(xy 77.47 69.85) (xy 72.39 69.85)
+			(xy 156.21 50.8) (xy 160.02 50.8)
 		)
 		(stroke
@@
 	(wire
 		(pts
-			(xy 130.81 64.77) (xy 130.81 62.23)
+			(xy 77.47 69.85) (xy 72.39 69.85)
 		)
 		(stroke
 			(width 0)
 			(type default)
-			(color 0 160 255 1)
 		)
 	)
 	(wire
 		(pts
-			(xy 80.01 46.99) (xy 85.09 46.99)
+			(xy 130.81 64.77) (xy 130.81 62.23)
 		)
 		(stroke
@@
 	(wire
 		(pts
-			(xy 130.81 41.91) (xy 125.73 41.91)
+			(xy 80.01 46.99) (xy 85.09 46.99)
 		)
 		(stroke
@@
 	(wire
 		(pts
-			(xy 123.19 36.83) (xy 125.73 36.83)
+			(xy 127 36.83) (xy 130.81 36.83)
 		)
 		(stroke
@@
 	(wire
 		(pts
-			(xy 114.3 36.83) (xy 118.11 36.83)
+			(xy 114.3 36.83) (xy 116.84 36.83)
 		)
 		(stroke
@@
 	(wire
 		(pts
+			(xy 116.84 36.83) (xy 121.92 36.83)
+		)
+		(stroke
+			(width 0)
+			(type default)
+			(color 255 0 0 1)
+		)
+	)
+	(wire
+		(pts
 			(xy 83.82 74.93) (xy 83.82 78.74)
 		)
@@
 	(wire
 		(pts
-			(xy 125.73 46.99) (xy 123.19 46.99)
+			(xy 127 46.99) (xy 130.81 46.99)
 		)
 		(stroke
@@
 	(wire
 		(pts
+			(xy 116.84 46.99) (xy 121.92 46.99)
+		)
+		(stroke
+			(width 0)
+			(type default)
+			(color 0 160 255 1)
+		)
+	)
+	(wire
+		(pts
 			(xy 151.13 68.58) (xy 156.21 68.58)
 		)
@@
 	(wire
 		(pts
-			(xy 114.3 46.99) (xy 118.11 46.99)
+			(xy 114.3 46.99) (xy 116.84 46.99)
 		)
 		(stroke
@@
 	(symbol
 		(lib_id "Device:R_Small")
-		(at 120.65 36.83 270)
+		(at 124.46 36.83 270)
 		(mirror x)
 		(unit 1)
@@
 		(dnp no)
 		(property "Reference" "R6"
-			(at 119.634 34.798 90)
+			(at 123.444 34.798 90)
 			(effects
 				(font
@@
 		)
 		(property "Value" "100"
-			(at 118.618 36.83 90)
+			(at 122.428 36.83 90)
 			(effects
 				(font
@@
 		)
 		(property "Footprint" "PCM_Resistor_THT_AKL:R_Axial_DIN0204_L3.6mm_D1.6mm_P7.62mm_Horizontal"
-			(at 120.65 36.83 0)
+			(at 124.46 36.83 0)
 			(effects
 				(font
@@
 		)
 		(property "Datasheet" "~"
-			(at 120.65 36.83 0)
+			(at 124.46 36.83 0)
 			(effects
 				(font
@@
 		)
 		(property "Description" "Resistor, small symbol"
-			(at 120.65 36.83 0)
+			(at 124.46 36.83 0)
 			(effects
 				(font
@@
 	(symbol
 		(lib_id "Device:R_Small")
-		(at 120.65 46.99 270)
+		(at 124.46 46.99 270)
 		(mirror x)
 		(unit 1)
@@
 		(dnp no)
 		(property "Reference" "R5"
-			(at 119.38 44.958 90)
+			(at 123.19 44.958 90)
 			(effects
 				(font
@@
 		)
 		(property "Value" "100"
-			(at 118.872 46.99 90)
+			(at 122.682 46.99 90)
 			(effects
 				(font
@@
 		)
 		(property "Footprint" "PCM_Resistor_THT_AKL:R_Axial_DIN0204_L3.6mm_D1.6mm_P7.62mm_Horizontal"
-			(at 120.65 46.99 0)
+			(at 124.46 46.99 0)
 			(effects
 				(font
@@
 		)
 		(property "Datasheet" "~"
-			(at 120.65 46.99 0)
+			(at 124.46 46.99 0)
 			(effects
 				(font
@@
 		)
 		(property "Description" "Resistor, small symbol"
-			(at 120.65 46.99 0)
+			(at 124.46 46.99 0)
 			(effects
 				(font
@@
 	(symbol
 		(lib_id "Device:C_Polarized_Small")
-		(at 125.73 44.45 180)
+		(at 116.84 44.45 180)
 		(unit 1)
 		(exclude_from_sim no)
@@
 		(fields_autoplaced yes)
 		(property "Reference" "C4"
-			(at 128.27 44.996 0)
+			(at 119.38 44.996 0)
 			(effects
 				(font
@@
 		)
 		(property "Value" "2200uF"
-			(at 123.19 43.7262 0)
+			(at 114.3 43.7262 0)
 			(effects
 				(font
@@
 		)
 		(property "Footprint" "Capacitor_THT:CP_Radial_D10.0mm_P5.00mm"
-			(at 125.73 44.45 0)
+			(at 116.84 44.45 0)
 			(effects
 				(font
@@
 		)
 		(property "Datasheet" "~"
-			(at 125.73 44.45 0)
+			(at 116.84 44.45 0)
 			(effects
 				(font
@@
 		)
 		(property "Description" "Polarized capacitor, small symbol"
-			(at 125.73 44.45 0)
+			(at 116.84 44.45 0)
 			(effects
 				(font
@@
 	(symbol
 		(lib_id "Device:C_Polarized_Small")
-		(at 125.73 39.37 0)
+		(at 116.84 39.37 0)
 		(unit 1)
 		(exclude_from_sim no)
@@
 		(fields_autoplaced yes)
 		(property "Reference" "C5"
-			(at 128.27 38.8238 0)
+			(at 119.38 38.8238 0)
 			(effects
 				(font
@@
 		)
 		(property "Value" "2200uF"
-			(at 123.19 40.0938 0)
+			(at 114.3 40.0938 0)
 			(effects
 				(font
@@
 		)
 		(property "Footprint" "Capacitor_THT:CP_Radial_D10.0mm_P5.00mm"
-			(at 125.73 39.37 0)
+			(at 116.84 39.37 0)
 			(effects
 				(font
@@
 		)
 		(property "Datasheet" "~"
-			(at 125.73 39.37 0)
+			(at 116.84 39.37 0)
 			(effects
 				(font
@@
 		)
 		(property "Description" "Polarized capacitor, small symbol"
-			(at 125.73 39.37 0)
+			(at 116.84 39.37 0)
 			(effects
 				(font

Commit message: changed resistors pin pitch from 7 to 5, compressed the board more
readme to be updated
Parts:
- J3: value -Gain+ -> +Gain-
- R1, R2, R3, R4, R5, R6, R7, R8: footprint PCM_Resistor_THT_AKL:R_Axial_DIN0204_L3.6mm_D1.6mm_P7.62mm_Horizontal -> PCM_Resistor_THT_AKL:R_Axial_DIN0204_L3.6mm_D1.6mm_P5.08mm_Horizontal
Changed lines of the file:
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@@
 			)
 		)
-		(property "Footprint" "PCM_Resistor_THT_AKL:R_Axial_DIN0204_L3.6mm_D1.6mm_P7.62mm_Horizontal"
+		(property "Footprint" "PCM_Resistor_THT_AKL:R_Axial_DIN0204_L3.6mm_D1.6mm_P5.08mm_Horizontal"
 			(at 81.28 91.44 0)
 			(effects
@@
 			)
 		)
-		(property "Footprint" "PCM_Resistor_THT_AKL:R_Axial_DIN0204_L3.6mm_D1.6mm_P7.62mm_Horizontal"
+		(property "Footprint" "PCM_Resistor_THT_AKL:R_Axial_DIN0204_L3.6mm_D1.6mm_P5.08mm_Horizontal"
 			(at 124.46 67.31 0)
 			(effects
@@
 			)
 		)
-		(property "Footprint" "PCM_Resistor_THT_AKL:R_Axial_DIN0204_L3.6mm_D1.6mm_P7.62mm_Horizontal"
+		(property "Footprint" "PCM_Resistor_THT_AKL:R_Axial_DIN0204_L3.6mm_D1.6mm_P5.08mm_Horizontal"
 			(at 124.46 36.83 0)
 			(effects
@@
 			)
 		)
-		(property "Footprint" "PCM_Resistor_THT_AKL:R_Axial_DIN0204_L3.6mm_D1.6mm_P7.62mm_Horizontal"
+		(property "Footprint" "PCM_Resistor_THT_AKL:R_Axial_DIN0204_L3.6mm_D1.6mm_P5.08mm_Horizontal"
 			(at 81.28 86.36 0)
 			(effects
@@
 			)
 		)
-		(property "Value" "-Gain+"
+		(property "Value" "+Gain-"
 			(at 147.32 50.546 0)
 			(effects
@@
 			)
 		)
-		(property "Footprint" "PCM_Resistor_THT_AKL:R_Axial_DIN0204_L3.6mm_D1.6mm_P7.62mm_Horizontal"
+		(property "Footprint" "PCM_Resistor_THT_AKL:R_Axial_DIN0204_L3.6mm_D1.6mm_P5.08mm_Horizontal"
 			(at 124.46 46.99 0)
 			(effects
@@
 			)
 		)
-		(property "Footprint" "PCM_Resistor_THT_AKL:R_Axial_DIN0204_L3.6mm_D1.6mm_P7.62mm_Horizontal"
+		(property "Footprint" "PCM_Resistor_THT_AKL:R_Axial_DIN0204_L3.6mm_D1.6mm_P5.08mm_Horizontal"
 			(at 130.81 67.31 0)
 			(effects
@@
 			)
 		)
-		(property "Footprint" "PCM_Resistor_THT_AKL:R_Axial_DIN0204_L3.6mm_D1.6mm_P7.62mm_Horizontal"
+		(property "Footprint" "PCM_Resistor_THT_AKL:R_Axial_DIN0204_L3.6mm_D1.6mm_P5.08mm_Horizontal"
 			(at 80.01 66.04 0)
 			(effects
@@
 			)
 		)
-		(property "Footprint" "PCM_Resistor_THT_AKL:R_Axial_DIN0204_L3.6mm_D1.6mm_P7.62mm_Horizontal"
+		(property "Footprint" "PCM_Resistor_THT_AKL:R_Axial_DIN0204_L3.6mm_D1.6mm_P5.08mm_Horizontal"
 			(at 80.01 78.74 0)
 			(effects

Commit message: changed footprints to 0805 smds, rewrote the readme
Parts:
- C1, C2, C3: footprint Capacitor_THT:C_Disc_D7.5mm_W2.5mm_P5.00mm -> Capacitor_SMD:C_0805_2012Metric
- R1, R2, R3, R4, R5, R6, R7, R8: footprint PCM_Resistor_THT_AKL:R_Axial_DIN0204_L3.6mm_D1.6mm_P5.08mm_Horizontal -> PCM_Resistor_SMD_AKL:R_0805_2012Metric
Changed lines of the file:
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@@
 		(dnp no)
 		(property "Reference" "R3"
-			(at 81.28 92.456 0)
+			(at 79.756 93.218 90)
 			(effects
 				(font
@@
 			)
 		)
-		(property "Footprint" "PCM_Resistor_THT_AKL:R_Axial_DIN0204_L3.6mm_D1.6mm_P5.08mm_Horizontal"
+		(property "Footprint" "PCM_Resistor_SMD_AKL:R_0805_2012Metric"
 			(at 81.28 91.44 0)
 			(effects
@@
 			)
 		)
-		(property "Footprint" "PCM_Resistor_THT_AKL:R_Axial_DIN0204_L3.6mm_D1.6mm_P5.08mm_Horizontal"
+		(property "Footprint" "PCM_Resistor_SMD_AKL:R_0805_2012Metric"
 			(at 124.46 67.31 0)
 			(effects
@@
 			)
 		)
-		(property "Footprint" "PCM_Resistor_THT_AKL:R_Axial_DIN0204_L3.6mm_D1.6mm_P5.08mm_Horizontal"
+		(property "Footprint" "PCM_Resistor_SMD_AKL:R_0805_2012Metric"
 			(at 124.46 36.83 0)
 			(effects
@@
 			)
 		)
-		(property "Footprint" "Capacitor_THT:C_Disc_D7.5mm_W2.5mm_P5.00mm"
+		(property "Footprint" "Capacitor_SMD:C_0805_2012Metric"
 			(at 80.01 74.93 0)
 			(effects
@@
 		(dnp no)
 		(property "Reference" "R4"
-			(at 81.026 85.344 0)
+			(at 82.55 88.138 90)
 			(effects
 				(font
@@
 			)
 		)
-		(property "Footprint" "PCM_Resistor_THT_AKL:R_Axial_DIN0204_L3.6mm_D1.6mm_P5.08mm_Horizontal"
+		(property "Footprint" "PCM_Resistor_SMD_AKL:R_0805_2012Metric"
 			(at 81.28 86.36 0)
 			(effects
@@
 			)
 		)
-		(property "Footprint" "Capacitor_THT:C_Disc_D7.5mm_W2.5mm_P5.00mm"
+		(property "Footprint" "Capacitor_SMD:C_0805_2012Metric"
 			(at 119.38 73.66 0)
 			(effects
@@
 			)
 		)
-		(property "Footprint" "Capacitor_THT:C_Disc_D7.5mm_W2.5mm_P5.00mm"
+		(property "Footprint" "Capacitor_SMD:C_0805_2012Metric"
 			(at 80.01 69.85 0)
 			(effects
@@
 			)
 		)
-		(property "Footprint" "PCM_Resistor_THT_AKL:R_Axial_DIN0204_L3.6mm_D1.6mm_P5.08mm_Horizontal"
+		(property "Footprint" "PCM_Resistor_SMD_AKL:R_0805_2012Metric"
 			(at 124.46 46.99 0)
 			(effects
@@
 			)
 		)
-		(property "Footprint" "PCM_Resistor_THT_AKL:R_Axial_DIN0204_L3.6mm_D1.6mm_P5.08mm_Horizontal"
+		(property "Footprint" "PCM_Resistor_SMD_AKL:R_0805_2012Metric"
 			(at 130.81 67.31 0)
 			(effects
@@
 			)
 		)
-		(property "Footprint" "PCM_Resistor_THT_AKL:R_Axial_DIN0204_L3.6mm_D1.6mm_P5.08mm_Horizontal"
+		(property "Footprint" "PCM_Resistor_SMD_AKL:R_0805_2012Metric"
 			(at 80.01 66.04 0)
 			(effects
@@
 			)
 		)
-		(property "Footprint" "PCM_Resistor_THT_AKL:R_Axial_DIN0204_L3.6mm_D1.6mm_P5.08mm_Horizontal"
+		(property "Footprint" "PCM_Resistor_SMD_AKL:R_0805_2012Metric"
 			(at 80.01 78.74 0)
 			(effects
